File: DP83848C-EvalBoard.kicad_pcb (KiCad board)
At the start: 4 copper layers, 75 x 100 mm, 186 parts, among them J1 Conn_01x02, J10 Conn_02x04_Odd_Even, J11 Conn_02x04_Odd_Even, J12 Conn_02x04_Odd_Even, J13 Conn_02x04_Odd_Even, J14 Conn_02x04_Odd_Even, J2 RJ45_LED_Shielded, J3 USB_C_Receptacle_USB2.0, J4 Conn_02x05_Odd_Even, J5 Conn_01x04, J6 Conn_01x04, J7 Conn_01x04, J8 Conn_02x08_Odd_Even, J9 Conn_02x08_Odd_Even, Q1 AO3401A, Q2 AO3400A, Q3 AO3401A, SW1 SW_Push, T1 H1102NL, U1 AMS1117-3.3, U10 CM1224, U11 CM1224, U12 CM1224, U13 CM1224, U14 CM1224, U15 CM1224, U2 DP83848C, U3 STM32F407VGTx, U4 USBLC6-2SC6, U5 CM1224, U6 CM1224, U7 CM1224, U8 CM1224, U9 CM1224, X1 50MHz, Y1 25MHz

Commit message: Layout
Parts:
- moved JP1 2.61 mm to (82.5, 90.0)
- moved R4 2.61 mm to (82.5, 95.0)
- moved JP2 2.24 mm to (94.0, 66.7)
- moved R30 2.24 mm to (94.0, 64.2)
- moved R31 2.24 mm to (94.0, 74.2)
- moved R39 1.35 mm to (79.0, 91.5), turned to 180 degrees
- moved R48 1.35 mm to (79.0, 86.2), turned to 180 degrees
- moved R44 1.12 mm to (79.0, 89.0), turned to 180 degrees
Routing:
- net /PHY/MII_MODE: track 8.92 -> 12.8 mm
- net /PHY/~RESET: track 8.31 -> 11.5 mm
- net GND: track 85.0 -> 85.6 mm, vias 69 -> 70
Other:
- board text added: "AN0 AN1 AN_EN Auto-Negotiation 0 0 0 10M HD forced 1 0 0 10M FD forced 0 1 0 100M HD forced 1 1 0 100M FD forced 0 0 1 10M H/FD advert. 1 0 1 100M H/FD advert. 0 1 1 10/100M HD advert. 1 1 1 10/100M H/FD advert."
- board text added: "AN_EN"
- board text added: "AUTO-NEG."
- board text added: "MII_MODE"
- board text added: "SNI_MODE"

Commit message: Update
Parts:
- removed JP2, JP3: Conn_01x03, Connector_PinHeader_2.54mm:PinHeader_1x03_P2.54mm_Vertical
- removed R17, R8: 33, Resistor_SMD:R_0402_1005Metric
- removed R31, R32, R33: 2.2k, Resistor_SMD:R_0402_1005Metric
- added G***: LOGO, ak:lemonhead, F.Cu at (71.2, 64.2)
- added G***: LOGO, ak:fluxcap, B.Cu at (75.0, 127.5)
- moved R30 14.3 mm to (91.2, 78.2)
- moved R57 1.12 mm to (73.0, 105.8)
- moved C24 0.50 mm to (70.8, 106.3)
- moved C29 0.50 mm to (67.4, 106.2)
- moved C30 0.50 mm to (68.4, 106.2)
- moved L1 0.50 mm to (66.0, 105.5)
- moved R49 0.50 mm to (69.4, 106.2)
Connections:
- R30 pad 2: Net-(JP2-Pad1) -> /PHY/MII_MODE
- U2 pad 39: Net-(R17-Pad1) -> /PHY/MII_MODE
- U2 pad 6: Net-(R8-Pad1) -> (no net)
Routing:
- net GND: track 85.6 -> 112.8 mm, vias 70 -> 86
- net /PHY/MII_MODE: track 12.8 -> 2.52 mm
- net /PHY/SNI_MODE: track 2.93 -> 0.00 mm
- net Net-(JP3-Pad1): track 2.71 -> 0.00 mm
- net Net-(JP2-Pad3): track 2.67 -> 0.00 mm
- net Net-(JP2-Pad1): track 2.67 -> 0.00 mm
- net Net-(JP3-Pad3): track 2.63 -> 0.00 mm
- net Net-(R17-Pad1): track 2.52 -> 0.00 mm
- net Net-(R8-Pad1): track 2.18 -> 0.00 mm
- net /ETH_MDC: track 39.4 -> 40.9 mm
- net /MCU/OSC_OUT: track 2.06 -> 2.98 mm
- net Net-(C32-Pad1): track 4.19 -> 3.61 mm
- net +3V3: track 86.4 -> 86.1 mm, vias 46 -> 45
Other:
- board text added: ""Quarantine edition""
- board text added: "100 Mbps"
- board text added: "DP83848C + STM32F407 Evaluation Board 12/2020 - Rev. A"
- board text added: "Made by Lemonhead"
- board text removed: "MII_MODE"
- board text removed: "SNI_MODE"

Commit message: DRC and minor changes
Parts:
- removed R15: 33, Resistor_SMD:R_0402_1005Metric
- C1: footprint Capacitor_SMD:C_Elec_6.3x7.7 -> Capacitor_SMD:C_Elec_6.3x5.8
- C18, C21: footprint Capacitor_SMD:C_0402_1005Metric -> Capacitor_SMD:C_0603_1608Metric
- moved C2 0.75 mm to (64.5, 149.8)
- moved C8 0.75 mm to (91.2, 79.5)
- moved C18 0.50 mm to (63.5, 122.0)
- moved C21 0.50 mm to (79.5, 127.0)
- moved G*** 0.35 mm to (71.5, 64.0)
- moved R11 0.25 mm to (91.2, 76.5)
- moved R12 0.25 mm to (91.2, 75.5)
- moved R18 0.25 mm to (91.2, 77.5)
- moved R30 0.25 mm to (91.2, 78.5)
Connections:
- U2 pad 38: Net-(R15-Pad1) -> (no net)
Routing:
- net GND: track 112.8 -> 109.3 mm
- net Net-(R15-Pad1): track 2.18 -> 0.00 mm
- net /ETH_TX_EN: track 69.1 -> 68.5 mm
- net /MCU/SWDIO: track 31.2 -> 31.8 mm
- net +3V3: track 86.1 -> 85.7 mm, vias 45 -> 66
- added copper zone on F.Cu, net GND
- removed copper zone on B.Cu, net Earth
- removed copper zone on B.Cu, net GND

Commit message: Minor changes
Parts:
- moved G*** 70.7 mm to (84.5, 133.5)
Routing:
- net +3V3: vias 66 -> 61
Other:
- board text added: ""Lockdown edition""
- board text removed: ""Quarantine edition""

Commit message: Minor changes and production files
Parts:
- added REF**: JLCPCB Tooling Hole, ak:JLCPCB Tooling Hole, F.Cu at (51.0, 153.0)
- added REF**: JLCPCB Tooling Hole, ak:JLCPCB Tooling Hole, F.Cu at (104.5, 153.0)
- added REF**: JLCPCB Tooling Hole, ak:JLCPCB Tooling Hole, F.Cu at (104.5, 59.5)
- added REF**: JLCPCB Tooling Hole, ak:JLCPCB Tooling Hole, F.Cu at (51.0, 59.5)
- C1: value 47uF -> 22uF; footprint Capacitor_SMD:C_Elec_6.3x5.8 -> Capacitor_Tantalum_SMD:CP_EIA-3528-15_AVX-H
- C2: value 100uF -> 22uF
- C31, C32: value TBD -> 18pF
- D3: value YL -> YE
- F1: value 200mA -> 500mA
- Q2: value AO3400A -> 2N7002
- R100, R101: value 4k7 -> 4.7k
- R49: value 0R -> 0
- Y1: value 25MHz -> 25MHz, 10ppm, 12pF
- moved C1 1.00 mm to (60.8, 142.5)
Connections:
- J3 pad S1: Net-(J3-PadS1) -> Earth
Routing:
- net GND: track 109.3 -> 101.9 mm, vias 86 -> 84
- net Earth: vias 5 -> 139
- added copper zone on B.Cu, net Earth
Other:
- rule pad_to_mask_clearance: 0.05 -> 0
