File: PHY.sch (KiCad schematic (older format))
At the start: 60 parts, among them J2 RJ45_LED_Shielded, T1 H1102NL, U2 DP83848C, X1 50MHz

Commit message: DRC and minor changes
Parts:
- removed R15: 33, Resistor_SMD:R_0402_1005Metric, symbol Device:R_Small
- C11, C12, C13, C14, C15, C3, C5, C6, C7, C8, C9: LCSC (none) -> C1525
- C16: LCSC (none) -> C23967
- D3: value YL -> YE; LCSC (none) -> C72038
- R10, R11, R12, R13, R14, R18, R42, R45, R46, R5, R6: LCSC (none) -> C25105
- R19, R21, R22, R30, R38, R39, R4, R43, R44, R47, R48: LCSC (none) -> C25879
- R20: LCSC (none) -> C17168
- R23, R24, R25, R26: LCSC (none) -> C25120
- R27: LCSC (none) -> C25900
- R28: LCSC (none) -> C25082
- R29: LCSC (none) -> C25092
- R34, R35, R36, R37: LCSC (none) -> C25133
- R40, R41: LCSC (none) -> C17888
- T1: LCSC (none) -> C18584
- U2: LCSC (none) -> C16688
Connections:
- no-connect marks 10 -> 11

Commit message: Minor changes
Parts:
- J2: Manufacturer (none) -> RJHSE-5381; Mouser (none) -> 523-RJHSE-5381
Changed lines of the file:
@@
 F 2 "Connector_RJ:RJ45_Amphenol_RJHSE538X" V 9450 2375 50  0001 C CNN
 F 3 "~" V 9450 2375 50  0001 C CNN
+F 4 "RJHSE-5381" H 9450 2350 50  0001 C CNN "Manufacturer"
+F 5 "523-RJHSE-5381" H 9450 2350 50  0001 C CNN "Mouser"
 	1    9450 2350
 	-1   0    0    1
