File: IO.sch (KiCad schematic (older format))
At the start: 63 parts, among them J10 Conn_02x04_Odd_Even, J11 Conn_02x04_Odd_Even, J12 Conn_02x04_Odd_Even, J13 Conn_02x04_Odd_Even, J14 Conn_02x04_Odd_Even, J5 Conn_01x04, J6 Conn_01x04, J7 Conn_01x04, J8 Conn_02x08_Odd_Even, J9 Conn_02x08_Odd_Even, U10 CM1224, U11 CM1224, U12 CM1224, U13 CM1224, U14 CM1224, U15 CM1224, U5 CM1224, U6 CM1224, U7 CM1224, U8 CM1224, U9 CM1224

Commit message: Layout
Parts:
- R100, R101, R62, R63, R64, R65, R66, R67, R68, R69: footprint Resistor_SMD:R_0603_1608Metric -> Resistor_SMD:R_0402_1005Metric
Connections:
- net ADC0_R: now also U11.3 (IO2); no longer U11.1 (IO1)
- net ADC1_R: now also U11.1 (IO1); no longer U11.3 (IO2)
- net ADC6_R: now also U15.6 (IO4); no longer U15.4 (IO3)
- net ADC7_R: now also U15.4 (IO3); no longer U15.6 (IO4)
- net GPIO0_R: now also U5.3 (IO2); no longer U5.1 (IO1)
- net GPIO1_R: now also U5.1 (IO1); no longer U5.3 (IO2)
- net I2C1_SCL_R: now also U13.3 (IO2); no longer U13.1 (IO1)
- net I2C1_SDA_R: now also U13.1 (IO1); no longer U13.3 (IO2)
- net SPI1_MISO_R: now also U6.3 (IO2); no longer U6.1 (IO1)
- net SPI1_MOSI_R: now also U6.1 (IO1); no longer U6.3 (IO2)
- net SPI1_NSS: no longer J11.7 (Pin_7), R85.1, U6.6 (IO4)
- net SPI1_SCK_R: now also U6.6 (IO4); no longer U6.4 (IO3)
- net USART1_RX_R: now also U7.4 (IO3); no longer U7.3 (IO2)
- net USART1_TX_R: now also U10.3 (IO2); no longer U7.1 (IO1)
- net USART2_TX_R: now also U10.1 (IO1); no longer U7.4 (IO3)
- net USART3_RX_R: now also U7.3 (IO2); no longer U10.3 (IO2)
- net USART3_TX_R: now also U7.1 (IO1); no longer U10.1 (IO1)
- new net SPI1_NSS_R: J11.7 (Pin_7), R85.1, U6.4 (IO3)
Changed lines of the file:
@@
 F 0 "R62" V 2050 900 50  0000 C CNN
 F 1 "33" V 2050 600 50  0000 C CNN
-F 2 "Resistor_SMD:R_0603_1608Metric" H 2100 750 50  0001 C CNN
+F 2 "Resistor_SMD:R_0402_1005Metric" H 2100 750 50  0001 C CNN
 F 3 "~" H 2100 750 50  0001 C CNN
 	1    2100 750
@@
 F 0 "R63" V 2050 1000 50  0000 C CNN
 F 1 "33" V 2050 700 50  0000 C CNN
-F 2 "Resistor_SMD:R_0603_1608Metric" H 2100 850 50  0001 C CNN
+F 2 "Resistor_SMD:R_0402_1005Metric" H 2100 850 50  0001 C CNN
 F 3 "~" H 2100 850 50  0001 C CNN
 	1    2100 850
@@
 F 0 "R64" V 2050 1100 50  0000 C CNN
 F 1 "33" V 2050 800 50  0000 C CNN
-F 2 "Resistor_SMD:R_0603_1608Metric" H 2100 950 50  0001 C CNN
+F 2 "Resistor_SMD:R_0402_1005Metric" H 2100 950 50  0001 C CNN
 F 3 "~" H 2100 950 50  0001 C CNN
 	1    2100 950
@@
 F 0 "R65" V 2050 1200 50  0000 C CNN
 F 1 "33" V 2050 900 50  0000 C CNN
-F 2 "Resistor_SMD:R_0603_1608Metric" H 2100 1050 50  0001 C CNN
+F 2 "Resistor_SMD:R_0402_1005Metric" H 2100 1050 50  0001 C CNN
 F 3 "~" H 2100 1050 50  0001 C CNN
 	1    2100 1050
@@
 F 0 "R66" V 2050 1300 50  0000 C CNN
 F 1 "33" V 2050 1000 50  0000 C CNN
-F 2 "Resistor_SMD:R_0603_1608Metric" H 2100 1150 50  0001 C CNN
+F 2 "Resistor_SMD:R_0402_1005Metric" H 2100 1150 50  0001 C CNN
 F 3 "~" H 2100 1150 50  0001 C CNN
 	1    2100 1150
@@
 F 0 "R67" V 2050 1400 50  0000 C CNN
 F 1 "33" V 2050 1100 50  0000 C CNN
-F 2 "Resistor_SMD:R_0603_1608Metric" H 2100 1250 50  0001 C CNN
+F 2 "Resistor_SMD:R_0402_1005Metric" H 2100 1250 50  0001 C CNN
 F 3 "~" H 2100 1250 50  0001 C CNN
 	1    2100 1250
@@
 F 0 "R68" V 2050 1500 50  0000 C CNN
 F 1 "33" V 2050 1200 50  0000 C CNN
-F 2 "Resistor_SMD:R_0603_1608Metric" H 2100 1350 50  0001 C CNN
+F 2 "Resistor_SMD:R_0402_1005Metric" H 2100 1350 50  0001 C CNN
 F 3 "~" H 2100 1350 50  0001 C CNN
 	1    2100 1350
@@
 F 0 "R69" V 2050 1600 50  0000 C CNN
 F 1 "33" V 2050 1300 50  0000 C CNN
-F 2 "Resistor_SMD:R_0603_1608Metric" H 2100 1450 50  0001 C CNN
+F 2 "Resistor_SMD:R_0402_1005Metric" H 2100 1450 50  0001 C CNN
 F 3 "~" H 2100 1450 50  0001 C CNN
 	1    2100 1450
@@
 Wire Wire Line
 	3600 1150 3250 1150
+Text Label 3250 1350 0    50   ~ 0
+GPIO0_R
 Text Label 3250 1150 0    50   ~ 0
-GPIO0_R
-Text Label 3250 1350 0    50   ~ 0
 GPIO1_R
 Wire Wire Line
@@
 	2000 3400 1300 3400
 Text Label 1800 3700 2    50   ~ 0
-SPI1_NSS
+SPI1_NSS_R
 Text Label 1800 3600 2    50   ~ 0
 SPI1_SCK_R
@@
 F 3 "~" H 2100 3600 50  0001 C CNN
 	1    2100 3600
-	0    -1   1    0
-$EndComp
-$Comp
-L Device:R_Small R?
-U 1 1 5FEF81D7
-P 2100 3700
-AR Path="/5FEF81D7" Ref="R?"  Part="1"
-AR Path="/5FEAD3F6/5FEF81D7" Ref="R85"  Part="1"
-F 0 "R85" V 2050 3850 50  0000 C CNN
-F 1 "33" V 2050 3550 50  0000 C CNN
-F 2 "Resistor_SMD:R_0402_1005Metric" H 2100 3700 50  0001 C CNN
-F 3 "~" H 2100 3700 50  0001 C CNN
-	1    2100 3700
 	0    -1   1    0
 $EndComp
@@
 Text HLabel 2400 6800 2    50   Input ~ 0
 USART3_RX
+Text Label 7150 1350 0    50   ~ 0
+ADC0_R
 Text Label 7150 1150 0    50   ~ 0
-ADC0_R
-Text Label 7150 1350 0    50   ~ 0
 ADC1_R
 Text Label 8850 1150 2    50   ~ 0
@@
 Text Label 9000 1350 0    50   ~ 0
 ADC5_R
+Text Label 10700 1350 2    50   ~ 0
+ADC6_R
 Text Label 10700 1150 2    50   ~ 0
-ADC6_R
-Text Label 10700 1350 2    50   ~ 0
 ADC7_R
+Text Label 5300 2550 2    50   ~ 0
+SPI1_NSS_R
 Text Label 5300 2750 2    50   ~ 0
-SPI1_NSS
-Text Label 5300 2550 2    50   ~ 0
 SPI1_SCK_R
+Text Label 3300 2550 0    50   ~ 0
+SPI1_MOSI_R
 Text Label 3300 2750 0    50   ~ 0
-SPI1_MOSI_R
-Text Label 3300 2550 0    50   ~ 0
 SPI1_MISO_R
 $Comp
@@
 	1    0    0    -1
 $EndComp
+Text Label 8000 4150 0    50   ~ 0
+I2C1_SCL_R
 Text Label 8000 3950 0    50   ~ 0
-I2C1_SCL_R
-Text Label 8000 4150 0    50   ~ 0
 I2C1_SDA_R
 $Comp
@@
 Wire Wire Line
 	6100 3950 5600 3950
-Text Label 5600 3950 0    50   ~ 0
-USART3_TX_R
+Wire Wire Line
+	4800 4150 5300 4150
+Wire Wire Line
+	5300 3950 4800 3950
+Wire Wire Line
+	3300 4150 3800 4150
+Wire Wire Line
+	3800 3950 3300 3950
 Text Label 5600 4150 0    50   ~ 0
-USART3_RX_R
-Wire Wire Line
-	4800 4150 5300 4150
-Wire Wire Line
-	5300 3950 4800 3950
-Text Label 5300 3950 2    50   ~ 0
-USART2_TX_R
-Text Label 5300 4150 2    50   ~ 0
-USART2_RX_R
-Wire Wire Line
-	3300 4150 3800 4150
-Wire Wire Line
-	3800 3950 3300 3950
-Text Label 3300 3950 0    50   ~ 0
 USART1_TX_R
-Text Label 3300 4150 0    50   ~ 0
-USART1_RX_R
 Text Label 9900 5600 2    50   ~ 0
 TMR4_R
@@
 F 0 "R101" V 4250 5800 50  0000 C CNN
 F 1 "4k7" V 4250 5500 50  0000 C CNN
-F 2 "Resistor_SMD:R_0603_1608Metric" H 4300 5650 50  0001 C CNN
+F 2 "Resistor_SMD:R_0402_1005Metric" H 4300 5650 50  0001 C CNN
 F 3 "~" H 4300 5650 50  0001 C CNN
 	1    4300 5650
@@
 F 0 "R100" V 4250 5500 50  0000 C CNN
 F 1 "4k7" V 4250 5200 50  0000 C CNN
-F 2 "Resistor_SMD:R_0603_1608Metric" H 4300 5350 50  0001 C CNN
+F 2 "Resistor_SMD:R_0402_1005Metric" H 4300 5350 50  0001 C CNN
 F 3 "~" H 4300 5350 50  0001 C CNN
 	1    4300 5350
@@
 U 1 1 60A53E4C
 P 4100 1250
+AR Path="/60A53E4C" Ref="U5"  Part="1"
+AR Path="/5FEAD3F6/60A53E4C" Ref="U5"  Part="1"
 F 0 "U5" H 4250 1700 50  0000 C CNN
 F 1 "CM1224" H 4350 800 50  0000 C CNN
@@
 U 1 1 60A5DBB6
 P 5950 1250
+AR Path="/60A5DBB6" Ref="U8"  Part="1"
+AR Path="/5FEAD3F6/60A5DBB6" Ref="U8"  Part="1"
 F 0 "U8" H 6100 1700 50  0000 C CNN
 F 1 "CM1224" H 6200 800 50  0000 C CNN
@@
 U 1 1 60A5ED6C
 P 8000 1250
+AR Path="/60A5ED6C" Ref="U11"  Part="1"
+AR Path="/5FEAD3F6/60A5ED6C" Ref="U11"  Part="1"
 F 0 "U11" H 8150 1700 50  0000 C CNN
 F 1 "CM1224" H 8250 800 50  0000 C CNN
@@
 U 1 1 60A608BF
 P 9850 1250
+AR Path="/60A608BF" Ref="U15"  Part="1"
+AR Path="/5FEAD3F6/60A608BF" Ref="U15"  Part="1"
 F 0 "U15" H 10000 1700 50  0000 C CNN
 F 1 "CM1224" H 10100 800 50  0000 C CNN
@@
 U 1 1 60A62C9E
 P 4300 2650
+AR Path="/60A62C9E" Ref="U6"  Part="1"
+AR Path="/5FEAD3F6/60A62C9E" Ref="U6"  Part="1"
 F 0 "U6" H 4450 3100 50  0000 C CNN
 F 1 "CM1224" H 4550 2200 50  0000 C CNN
@@
 U 1 1 60A658D9
 P 6600 2650
+AR Path="/60A658D9" Ref="U9"  Part="1"
+AR Path="/5FEAD3F6/60A658D9" Ref="U9"  Part="1"
 F 0 "U9" H 6750 3100 50  0000 C CNN
 F 1 "CM1224" H 6850 2200 50  0000 C CNN
@@
 U 1 1 60A67356
 P 9000 2650
+AR Path="/60A67356" Ref="U12"  Part="1"
+AR Path="/5FEAD3F6/60A67356" Ref="U12"  Part="1"
 F 0 "U12" H 9150 3100 50  0000 C CNN
 F 1 "CM1224" H 9250 2200 50  0000 C CNN
@@
 U 1 1 60A6A99A
 P 4300 4050
+AR Path="/60A6A99A" Ref="U7"  Part="1"
+AR Path="/5FEAD3F6/60A6A99A" Ref="U7"  Part="1"
 F 0 "U7" H 4450 4500 50  0000 C CNN
 F 1 "CM1224" H 4550 3600 50  0000 C CNN
@@
 U 1 1 60A6C09D
 P 6600 4050
+AR Path="/60A6C09D" Ref="U10"  Part="1"
+AR Path="/5FEAD3F6/60A6C09D" Ref="U10"  Part="1"
 F 0 "U10" H 6750 4500 50  0000 C CNN
 F 1 "CM1224" H 6850 3600 50  0000 C CNN
@@
 U 1 1 60A6D298
 P 9050 4050
+AR Path="/60A6D298" Ref="U13"  Part="1"
+AR Path="/5FEAD3F6/60A6D298" Ref="U13"  Part="1"
 F 0 "U13" H 9200 4500 50  0000 C CNN
 F 1 "CM1224" H 9300 3600 50  0000 C CNN
@@
 U 1 1 60A7334D
 P 9050 5500
+AR Path="/60A7334D" Ref="U14"  Part="1"
+AR Path="/5FEAD3F6/60A7334D" Ref="U14"  Part="1"
 F 0 "U14" H 9200 5950 50  0000 C CNN
 F 1 "CM1224" H 9300 5050 50  0000 C CNN
@@
 	1    0    0    -1
 $EndComp
+Text Label 5300 3950 2    50   ~ 0
+USART1_RX_R
+Text Label 3300 4150 0    50   ~ 0
+USART3_RX_R
+Text Label 5300 4150 2    50   ~ 0
+USART2_RX_R
+Text Label 5600 3950 0    50   ~ 0
+USART2_TX_R
+Text Label 3300 3950 0    50   ~ 0
+USART3_TX_R
+$Comp
+L Device:R_Small R?
+U 1 1 5FEF81D7
+P 2100 3700
+AR Path="/5FEF81D7" Ref="R?"  Part="1"
+AR Path="/5FEAD3F6/5FEF81D7" Ref="R85"  Part="1"
+F 0 "R85" V 2050 3850 50  0000 C CNN
+F 1 "33" V 2050 3550 50  0000 C CNN
+F 2 "Resistor_SMD:R_0402_1005Metric" H 2100 3700 50  0001 C CNN
+F 3 "~" H 2100 3700 50  0001 C CNN
+	1    2100 3700
+	0    -1   1    0
+$EndComp
 $EndSCHEMATC

Commit message: DRC and minor changes
Parts:
- R100, R101: value 4k7 -> 4.7k; LCSC (none) -> C25900
- R102, R103, R62, R63, R64, R65, R66, R67, R68, R69, R70, R71, R72, R73, R74, R75, R76, R77, R78, R79, R80, R81, R82, R83, R84, R85, R86, R87, R88, R89, R90, R91, R92, R93, R94, R95, R96, R97, R98, R99: LCSC (none) -> C25105
- U10, U11, U12, U13, U14, U15, U5, U6, U7, U8, U9: LCSC (none) -> CM1224
Connections:
- no-connect marks 0 -> 4

Commit message: Minor changes and production files
Parts:
- U10, U11, U12, U13, U14, U15, U5, U6, U7, U8, U9: LCSC CM1224 -> C233379
Changed lines of the file:
@@
 F 2 "Package_TO_SOT_SMD:SOT-23-6" H 4800 800 50  0001 C CNN
 F 3 "http://www.onsemi.com/pub/Collateral/SRV05-4-D.PDF" H 4100 1250 50  0001 C CNN
-F 4 "CM1224" H 4100 1250 50  0001 C CNN "LCSC"
+F 4 "C233379" H 4100 1250 50  0001 C CNN "LCSC"
 	1    4100 1250
 	1    0    0    -1
@@
 F 2 "Package_TO_SOT_SMD:SOT-23-6" H 6650 800 50  0001 C CNN
 F 3 "http://www.onsemi.com/pub/Collateral/SRV05-4-D.PDF" H 5950 1250 50  0001 C CNN
-F 4 "CM1224" H 5950 1250 50  0001 C CNN "LCSC"
+F 4 "C233379" H 5950 1250 50  0001 C CNN "LCSC"
 	1    5950 1250
 	1    0    0    -1
@@
 F 2 "Package_TO_SOT_SMD:SOT-23-6" H 8700 800 50  0001 C CNN
 F 3 "http://www.onsemi.com/pub/Collateral/SRV05-4-D.PDF" H 8000 1250 50  0001 C CNN
-F 4 "CM1224" H 8000 1250 50  0001 C CNN "LCSC"
+F 4 "C233379" H 8000 1250 50  0001 C CNN "LCSC"
 	1    8000 1250
 	1    0    0    -1
@@
 F 2 "Package_TO_SOT_SMD:SOT-23-6" H 10550 800 50  0001 C CNN
 F 3 "http://www.onsemi.com/pub/Collateral/SRV05-4-D.PDF" H 9850 1250 50  0001 C CNN
-F 4 "CM1224" H 9850 1250 50  0001 C CNN "LCSC"
+F 4 "C233379" H 9850 1250 50  0001 C CNN "LCSC"
 	1    9850 1250
 	1    0    0    -1
@@
 F 2 "Package_TO_SOT_SMD:SOT-23-6" H 5000 2200 50  0001 C CNN
 F 3 "http://www.onsemi.com/pub/Collateral/SRV05-4-D.PDF" H 4300 2650 50  0001 C CNN
-F 4 "CM1224" H 4300 2650 50  0001 C CNN "LCSC"
+F 4 "C233379" H 4300 2650 50  0001 C CNN "LCSC"
 	1    4300 2650
 	1    0    0    -1
@@
 F 2 "Package_TO_SOT_SMD:SOT-23-6" H 7300 2200 50  0001 C CNN
 F 3 "http://www.onsemi.com/pub/Collateral/SRV05-4-D.PDF" H 6600 2650 50  0001 C CNN
-F 4 "CM1224" H 6600 2650 50  0001 C CNN "LCSC"
+F 4 "C233379" H 6600 2650 50  0001 C CNN "LCSC"
 	1    6600 2650
 	1    0    0    -1
@@
 F 2 "Package_TO_SOT_SMD:SOT-23-6" H 9700 2200 50  0001 C CNN
 F 3 "http://www.onsemi.com/pub/Collateral/SRV05-4-D.PDF" H 9000 2650 50  0001 C CNN
-F 4 "CM1224" H 9000 2650 50  0001 C CNN "LCSC"
+F 4 "C233379" H 9000 2650 50  0001 C CNN "LCSC"
 	1    9000 2650
 	1    0    0    -1
@@
 F 2 "Package_TO_SOT_SMD:SOT-23-6" H 5000 3600 50  0001 C CNN
 F 3 "http://www.onsemi.com/pub/Collateral/SRV05-4-D.PDF" H 4300 4050 50  0001 C CNN
-F 4 "CM1224" H 4300 4050 50  0001 C CNN "LCSC"
+F 4 "C233379" H 4300 4050 50  0001 C CNN "LCSC"
 	1    4300 4050
 	1    0    0    -1
@@
 F 2 "Package_TO_SOT_SMD:SOT-23-6" H 7300 3600 50  0001 C CNN
 F 3 "http://www.onsemi.com/pub/Collateral/SRV05-4-D.PDF" H 6600 4050 50  0001 C CNN
-F 4 "CM1224" H 6600 4050 50  0001 C CNN "LCSC"
+F 4 "C233379" H 6600 4050 50  0001 C CNN "LCSC"
 	1    6600 4050
 	1    0    0    -1
@@
 F 2 "Package_TO_SOT_SMD:SOT-23-6" H 9750 3600 50  0001 C CNN
 F 3 "http://www.onsemi.com/pub/Collateral/SRV05-4-D.PDF" H 9050 4050 50  0001 C CNN
-F 4 "CM1224" H 9050 4050 50  0001 C CNN "LCSC"
+F 4 "C233379" H 9050 4050 50  0001 C CNN "LCSC"
 	1    9050 4050
 	1    0    0    -1
@@
 F 2 "Package_TO_SOT_SMD:SOT-23-6" H 9750 5050 50  0001 C CNN
 F 3 "http://www.onsemi.com/pub/Collateral/SRV05-4-D.PDF" H 9050 5500 50  0001 C CNN
-F 4 "CM1224" H 9050 5500 50  0001 C CNN "LCSC"
+F 4 "C233379" H 9050 5500 50  0001 C CNN "LCSC"
 	1    9050 5500
 	1    0    0    -1
