File: MCU.sch (KiCad schematic (older format))
At the start: 33 parts

Commit message: Component placement
Parts:
- removed JP?: Conn_02x03_Counter_Clockwise, symbol Connector_Generic:Conn_02x03_Counter_Clockwise
- added F1: 200mA, Fuse:Fuse_1812_4532Metric_Castellated, symbol Device:Polyfuse_Small
- added J11: USB_C_Receptacle_USB2.0, ak:DX07S016JA3R1500, symbol Connector:USB_C_Receptacle_USB2.0
- added JP7: Conn_02x03_Odd_Even, Connector_PinHeader_2.54mm:PinHeader_2x03_P2.54mm_Vertical, symbol Connector_Generic:Conn_02x03_Odd_Even
- added L2: 100@100MHz, Inductor_SMD:L_0805_2012Metric, symbol Device:L_Small
- added R57, R58: 5.1k, Resistor_SMD:R_0402_1005Metric, symbol Device:R_Small
- added U4: USBLC6-2SC6, Package_TO_SOT_SMD:SOT-23-6, symbol Power_Protection:USBLC6-2SC6
- C17, C18, C19, C20, C21, C22, C23, C24, C25, C26, C27, C28, C29, C30, C31: renamed from C?; footprint (none) -> Capacitor_SMD:C_0402_1005Metric
- D4: renamed from D?; footprint (none) -> LED_SMD:LED_0603_1608Metric
- J12: renamed from J?; footprint (none) -> Connector_PinHeader_2.54mm:PinHeader_2x05_P2.54mm_Vertical
- L1: renamed from L?; footprint (none) -> Inductor_SMD:L_0805_2012Metric
- R51, R52, R53, R54, R55, R56, R59, R60, R61, R62, R63: renamed from R?; footprint (none) -> Resistor_SMD:R_0402_1005Metric
- SW1: renamed from SW?; footprint (none) -> Button_Switch_THT:SW_PUSH_6mm
- Y1: renamed from Y?; footprint (none) -> Crystal:Crystal_SMD_3225-4Pin_3.2x2.5mm
- gave numbers to parts that had none: 1
Connections:
- net labels added: USB_CONN_D+, USB_CONN_D-, VUSB
- wire segments 202 -> 228
- no-connect marks 2 -> 5
Other:
- moved on the sheet: D4, R52

Commit message: Routing
Parts:
- added C32: 10uF, Capacitor_Tantalum_SMD:CP_EIA-3216-18_Kemet-A, symbol Device:CP_Small
Connections:
- net +3V3: now also C32.1
- net GND: now also C32.2
- net VREF+: now reaches R51.1, U3.21 (VREF+)
Other:
- moved on the sheet: C17, C20, C22, C23, C24, C25, C26, C27, C28, C29, L1, R51

Commit message: Added ESD protection
Parts:
- renumbered C32 to C17, C17 to C19, C19 to C20, C20 to C22, C22 to C23, C23 to C24, C24 to C25, C25 to C26, C26 to C27, C27 to C28, C28 to C29, C29 to C30, C30 to C31, C31 to C32, J11 to J3, J12 to J4, R51 to R49, R52 to R50, R53 to R51, R54 to R52, R55 to R53, R56 to R54, R57 to R55, R58 to R56, R59 to R57, R60 to R58, R61 to R59, R62 to R60, R63 to R61

Commit message: DRC and minor changes
Parts:
- C18, C21: footprint Capacitor_SMD:C_0402_1005Metric -> Capacitor_SMD:C_0603_1608Metric; LCSC (none) -> C23630
- C19: LCSC (none) -> C23733
- C20, C22, C23, C24, C25, C26, C27, C28, C30: LCSC (none) -> C1525
- C29: LCSC (none) -> C52923
- C31, C32: value TBD -> 18pF; LCSC (none) -> C1549
- D4: LCSC (none) -> C72041
- J3: symbol Connector:USB_C_Receptacle_USB2.0 -> DP83848C-EvalBoard-rescue:USB_C_Receptacle_USB2.0-Connector
- R49: value 0R -> 0; LCSC (none) -> C17168
- R50: LCSC (none) -> C25076
- R51, R52, R53, R54: LCSC (none) -> C25744
- R55, R56: LCSC (none) -> C25905
- R57: LCSC (none) -> C26083
- R58, R59, R60, R61: LCSC (none) -> C25105
- U3: LCSC (none) -> C28730
- U4: LCSC (none) -> C558442
- Y1: value 25MHz -> 25MHz, 10ppm, 12pF; LCSC (none) -> C9006
Connections:
- net ETH_REF_CLK: no longer names the net of U3.24 (PA1)
- no-connect marks 5 -> 30
Other:
- moved on the sheet: D4, R50

Commit message: Minor changes
Parts:
- F1: value 200mA -> 500mA; Manufacturer (none) -> 1812L050/60MR; Mouser (none) -> 576-1812L050/60MR
- J3: Manufacturer (none) -> DX07S016JA3R1500; Mouser (none) -> 656-DX07S016JA3R1500
- SW1: Manufacturer (none) -> PTS645SK432LFS; Mouser (none) -> 611-PTS645SK432
Changed lines of the file:
@@
 F 2 "Button_Switch_THT:SW_PUSH_6mm" H 1100 2350 50  0001 C CNN
 F 3 "~" H 1100 2350 50  0001 C CNN
+F 4 "PTS645SK432LFS" H 1100 2150 50  0001 C CNN "Manufacturer"
+F 5 "611-PTS645SK432" H 1100 2150 50  0001 C CNN "Mouser"
 	1    1100 2150
 	0    -1   1    0
@@
 F 2 "ak:DX07S016JA3R1500" H 7800 3550 50  0001 C CNN
 F 3 "https://www.usb.org/sites/default/files/documents/usb_type-c.zip" H 7800 3550 50  0001 C CNN
+F 4 "DX07S016JA3R1500 " H 7650 3550 50  0001 C CNN "Manufacturer"
+F 5 "656-DX07S016JA3R1500" H 7650 3550 50  0001 C CNN "Mouser"
 	1    7650 3550
 	1    0    0    -1
@@
 AR Path="/615282EA/5FF37565" Ref="F1"  Part="1"
 F 0 "F1" V 10395 2950 50  0000 C CNN
-F 1 "200mA" V 10486 2950 50  0000 C CNN
+F 1 "500mA" V 10486 2950 50  0000 C CNN
 F 2 "Fuse:Fuse_1812_4532Metric_Castellated" H 10650 2750 50  0001 L CNN
 F 3 "~" H 10600 2950 50  0001 C CNN
+F 4 "1812L050/60MR" H 10600 2950 50  0001 C CNN "Manufacturer"
+F 5 "576-1812L050/60MR" H 10600 2950 50  0001 C CNN "Mouser"
 	1    10600 2950
 	0    1    1    0

Commit message: Minor changes and production files
Parts:
- F1: LCSC (none) -> C516066
- U4: LCSC C558442 -> C7519
Connections:
- net Earth: now reaches J3.S1 (SHIELD)
- no-connect marks 30 -> 29
Changed lines of the file:
@@
 NoConn ~ 8250 4050
 NoConn ~ 8250 4150
-NoConn ~ 7350 4450
 $Comp
 L power:GND #PWR?
@@
 F 2 "Package_TO_SOT_SMD:SOT-23-6" H 10050 3100 50  0001 C CNN
 F 3 "https://www.st.com/resource/en/datasheet/usblc6-2.pdf" H 10250 3950 50  0001 C CNN
-F 4 "C558442" H 10050 3600 50  0001 C CNN "LCSC"
+F 4 "C7519" H 10050 3600 50  0001 C CNN "LCSC"
 	1    10050 3600
 	-1   0    0    -1
@@
 F 4 "1812L050/60MR" H 10600 2950 50  0001 C CNN "Manufacturer"
 F 5 "576-1812L050/60MR" H 10600 2950 50  0001 C CNN "Mouser"
+F 6 "C516066" H 10600 2950 50  0001 C CNN "LCSC"
 	1    10600 2950
 	0    1    1    0
@@
 Text Label 4800 3450 2    50   ~ 0
 USB_FS_D+
+$Comp
+L power:Earth #PWR0123
+U 1 1 603677B1
+P 7350 4450
+F 0 "#PWR0123" H 7350 4200 50  0001 C CNN
+F 1 "Earth" H 7350 4300 50  0001 C CNN
+F 2 "" H 7350 4450 50  0001 C CNN
+F 3 "~" H 7350 4450 50  0001 C CNN
+	1    7350 4450
+	1    0    0    -1
+$EndComp
 $EndSCHEMATC
