File: PSU.sch (KiCad schematic (older format))
At the start: 12 parts, among them J1 Conn_01x02, Q1 AO3401A, Q2 AO3400A, Q3 AO3401A, U1 AMS1117-3.3

Commit message: DRC and minor changes
Parts:
- C1: footprint Capacitor_SMD:C_Elec_6.3x7.7 -> Capacitor_SMD:C_Elec_6.3x5.8; LCSC (none) -> C178565
- C2: LCSC (none) -> C16133
- D1: LCSC (none) -> C72043
- D2: LCSC (none) -> C72038
- Q1, Q3: LCSC (none) -> C15127
- Q2: symbol Transistor_FET:AO3400A -> DP83848C-EvalBoard-rescue:AO3400A-Transistor_FET; LCSC (none) -> C20917
- R1, R3: LCSC (none) -> C25105
- R2: LCSC (none) -> C25792
- U1: LCSC (none) -> C6186
Changed lines of the file:
@@
 F 2 "Package_TO_SOT_SMD:SOT-223-3_TabPin2" H 7400 2400 50  0001 C CNN
 F 3 "http://www.advanced-monolithic.com/pdf/ds1117.pdf" H 7500 1950 50  0001 C CNN
+F 4 "C6186" H 7400 2200 50  0001 C CNN "LCSC"
 	1    7400 2200
 	1    0    0    -1
@@
 F 2 "Capacitor_Tantalum_SMD:CP_EIA-3528-15_AVX-H" H 7900 2400 50  0001 C CNN
 F 3 "~" H 7900 2400 50  0001 C CNN
+F 4 "C16133" H 7900 2400 50  0001 C CNN "LCSC"
 	1    7900 2400
 	1    0    0    -1
@@
 F 0 "C1" H 6938 2446 50  0000 L CNN
 F 1 "47uF" H 6938 2355 50  0000 L CNN
-F 2 "Capacitor_SMD:C_Elec_6.3x7.7" H 6850 2400 50  0001 C CNN
+F 2 "Capacitor_SMD:C_Elec_6.3x5.8" H 6850 2400 50  0001 C CNN
 F 3 "~" H 6850 2400 50  0001 C CNN
+F 4 "C178565" H 6850 2400 50  0001 C CNN "LCSC"
 	1    6850 2400
 	1    0    0    -1
@@
 F 2 "Resistor_SMD:R_0402_1005Metric" H 5000 2400 50  0001 C CNN
 F 3 "~" H 5000 2400 50  0001 C CNN
+F 4 "C25792" H 5000 2400 50  0001 C CNN "LCSC"
 	1    5000 2400
 	-1   0    0    -1
 $EndComp
 $Comp
-L Transistor_FET:AO3400A Q?
+L DP83848C-EvalBoard-rescue:AO3400A-Transistor_FET Q?
 U 1 1 61CE9BD4
 P 4900 2950
@@
 F 2 "Package_TO_SOT_SMD:SOT-23" H 5100 2875 50  0001 L CIN
 F 3 "http://www.aosmd.com/pdfs/datasheet/AO3400A.pdf" H 4900 2950 50  0001 L CNN
+F 4 "C20917" H 4900 2950 50  0001 C CNN "LCSC"
 	1    4900 2950
 	1    0    0    -1
@@
 F 2 "Package_TO_SOT_SMD:SOT-23" H 4850 2225 50  0001 L CIN
 F 3 "http://www.aosmd.com/pdfs/datasheet/AO3401A.pdf" H 4650 2300 50  0001 L CNN
+F 4 "C15127" H 4650 2300 50  0001 C CNN "LCSC"
 	1    4650 2300
 	0    -1   -1   0
@@
 F 2 "Package_TO_SOT_SMD:SOT-23" H 5550 2225 50  0001 L CIN
 F 3 "http://www.aosmd.com/pdfs/datasheet/AO3401A.pdf" H 5350 2300 50  0001 L CNN
+F 4 "C15127" H 5350 2300 50  0001 C CNN "LCSC"
 	1    5350 2300
 	0    1    -1   0
@@
 F 2 "LED_SMD:LED_0603_1608Metric" V 5650 2650 50  0001 C CNN
 F 3 "~" V 5650 2650 50  0001 C CNN
+F 4 "C72038" H 5650 2650 50  0001 C CNN "LCSC"
 	1    5650 2650
 	0    -1   -1   0
@@
 F 2 "Resistor_SMD:R_0402_1005Metric" H 5650 2400 50  0001 C CNN
 F 3 "~" H 5650 2400 50  0001 C CNN
+F 4 "C25105" H 5650 2400 50  0001 C CNN "LCSC"
 	1    5650 2400
 	-1   0    0    -1
@@
 F 2 "LED_SMD:LED_0603_1608Metric" V 4100 2650 50  0001 C CNN
 F 3 "~" V 4100 2650 50  0001 C CNN
+F 4 "C72043" H 4100 2650 50  0001 C CNN "LCSC"
 	1    4100 2650
 	0    -1   -1   0
@@
 F 2 "Resistor_SMD:R_0402_1005Metric" H 4100 2400 50  0001 C CNN
 F 3 "~" H 4100 2400 50  0001 C CNN
+F 4 "C25105" H 4100 2400 50  0001 C CNN "LCSC"
 	1    4100 2400
 	-1   0    0    -1
@@
 Wire Wire Line
 	4100 2200 4350 2200
+$Comp
+L power:+5V #PWR?
+U 1 1 6016C4CE
+P 6550 7300
+AR Path="/6016C4CE" Ref="#PWR?"  Part="1"
+AR Path="/61CDC1C0/6016C4CE" Ref="#PWR0120"  Part="1"
+F 0 "#PWR0120" H 6550 7150 50  0001 C CNN
+F 1 "+5V" H 6565 7473 50  0000 C CNN
+F 2 "" H 6550 7300 50  0001 C CNN
+F 3 "" H 6550 7300 50  0001 C CNN
+	1    6550 7300
+	-1   0    0    -1
+$EndComp
+$Comp
+L power:PWR_FLAG #FLG0102
+U 1 1 6016E2EF
+P 6550 7300
+F 0 "#FLG0102" H 6550 7375 50  0001 C CNN
+F 1 "PWR_FLAG" H 6550 7473 50  0000 C CNN
+F 2 "" H 6550 7300 50  0001 C CNN
+F 3 "~" H 6550 7300 50  0001 C CNN
+	1    6550 7300
+	-1   0    0    1
+$EndComp
+$Comp
+L power:GND #PWR?
+U 1 1 601704DB
+P 6150 7350
+AR Path="/601704DB" Ref="#PWR?"  Part="1"
+AR Path="/61CDC1C0/601704DB" Ref="#PWR0121"  Part="1"
+F 0 "#PWR0121" H 6150 7100 50  0001 C CNN
+F 1 "GND" H 6155 7177 50  0001 C CNN
+F 2 "" H 6150 7350 50  0001 C CNN
+F 3 "" H 6150 7350 50  0001 C CNN
+	1    6150 7350
+	-1   0    0    -1
+$EndComp
+$Comp
+L power:PWR_FLAG #FLG0103
+U 1 1 60170C26
+P 6150 7350
+F 0 "#FLG0103" H 6150 7425 50  0001 C CNN
+F 1 "PWR_FLAG" H 6150 7523 50  0000 C CNN
+F 2 "" H 6150 7350 50  0001 C CNN
+F 3 "~" H 6150 7350 50  0001 C CNN
+	1    6150 7350
+	1    0    0    -1
+$EndComp
 $EndSCHEMATC

Commit message: Minor changes
Parts:
- J1: Manufacturer (none) -> 22-11-2022; Mouser (none) -> 538-22-11-2022
Changed lines of the file:
@@
 F 2 "ak:Molex_022112022" H 3400 2200 50  0001 C CNN
 F 3 "~" H 3400 2200 50  0001 C CNN
+F 4 "22-11-2022" H 3400 2200 50  0001 C CNN "Manufacturer"
+F 5 "538-22-11-2022" H 3400 2200 50  0001 C CNN "Mouser"
 	1    3400 2200
 	-1   0    0    -1

Commit message: Minor changes and production files
Parts:
- removed Q2: AO3400A, Package_TO_SOT_SMD:SOT-23, symbol DP83848C-EvalBoard-rescue:AO3400A-Transistor_FET
- added Q2: 2N7002, Package_TO_SOT_SMD:SOT-23, symbol Transistor_FET:2N7002
- C1: value 47uF -> 22uF; footprint Capacitor_SMD:C_Elec_6.3x5.8 -> Capacitor_Tantalum_SMD:CP_EIA-3528-15_AVX-H; LCSC C178565 -> C8020
- C2: value 100uF -> 22uF; LCSC C16133 -> C8020
Connections:
- net GND: now also Q2.2 (S)
- net VEXT: now also Q2.1 (G)
- net at Q1.1 (G), R2.2: now also Q2.3 (D)
Changed lines of the file:
@@
 AR Path="/61CDC1C0/61CE9B79" Ref="C2"  Part="1"
 F 0 "C2" H 7988 2446 50  0000 L CNN
-F 1 "100uF" H 7988 2355 50  0000 L CNN
+F 1 "22uF" H 7988 2355 50  0000 L CNN
 F 2 "Capacitor_Tantalum_SMD:CP_EIA-3528-15_AVX-H" H 7900 2400 50  0001 C CNN
 F 3 "~" H 7900 2400 50  0001 C CNN
-F 4 "C16133" H 7900 2400 50  0001 C CNN "LCSC"
+F 4 "C8020" H 7900 2400 50  0001 C CNN "LCSC"
 	1    7900 2400
 	1    0    0    -1
@@
 AR Path="/61CDC1C0/61CE9B7F" Ref="C1"  Part="1"
 F 0 "C1" H 6938 2446 50  0000 L CNN
-F 1 "47uF" H 6938 2355 50  0000 L CNN
-F 2 "Capacitor_SMD:C_Elec_6.3x5.8" H 6850 2400 50  0001 C CNN
+F 1 "22uF" H 6938 2355 50  0000 L CNN
+F 2 "Capacitor_Tantalum_SMD:CP_EIA-3528-15_AVX-H" H 6850 2400 50  0001 C CNN
 F 3 "~" H 6850 2400 50  0001 C CNN
-F 4 "C178565" H 6850 2400 50  0001 C CNN "LCSC"
+F 4 "C8020" H 6850 2400 50  0001 C CNN "LCSC"
 	1    6850 2400
 	1    0    0    -1
@@
 	1    5000 2400
 	-1   0    0    -1
-$EndComp
-$Comp
-L DP83848C-EvalBoard-rescue:AO3400A-Transistor_FET Q?
-U 1 1 61CE9BD4
-P 4900 2950
-AR Path="/61CE9BD4" Ref="Q?"  Part="1"
-AR Path="/61CDC1C0/61CE9BD4" Ref="Q2"  Part="1"
-F 0 "Q2" H 5105 2996 50  0000 L CNN
-F 1 "AO3400A" H 5105 2905 50  0000 L CNN
-F 2 "Package_TO_SOT_SMD:SOT-23" H 5100 2875 50  0001 L CIN
-F 3 "http://www.aosmd.com/pdfs/datasheet/AO3400A.pdf" H 4900 2950 50  0001 L CNN
-F 4 "C20917" H 4900 2950 50  0001 C CNN "LCSC"
-	1    4900 2950
-	1    0    0    -1
 $EndComp
 Wire Wire Line
@@
 	1    0    0    -1
 $EndComp
+$Comp
+L Transistor_FET:2N7002 Q2
+U 1 1 60452E50
+P 4900 2950
+F 0 "Q2" H 5104 2996 50  0000 L CNN
+F 1 "2N7002" H 5104 2905 50  0000 L CNN
+F 2 "Package_TO_SOT_SMD:SOT-23" H 5100 2875 50  0001 L CIN
+F 3 "https://www.onsemi.com/pub/Collateral/NDS7002A-D.PDF" H 4900 2950 50  0001 L CNN
+F 4 "C8545" H 4900 2950 50  0001 C CNN "LCSC"
+	1    4900 2950
+	1    0    0    -1
+$EndComp
